Commit message: Add fanuc m20id35 to cage mockup

File: src/testbed/safe_energetics_testbed/urdf/irb6640_180_255.xacro (robot description, xacro)
@@ -1,4 +1,5 @@
 <?xml version="1.0" ?>
 <robot name="abb_irb6640_180_255" xmlns:xacro="http://ros.org/wiki/xacro">
+  <xacro:include filename="$(find fanuc_m20id35_support)/urdf/fanuc_common_materials.xacro"/>
   <xacro:include filename="$(find rpi_abb_irb6640_180_255_support)/urdf/irb6640_180_255_macro.xacro"/>
   <xacro:abb_irb6640_180_255 prefix="abb_"/>
@@ -9,5 +10,5 @@
         <box size="0.9144 0.9144 0.0254"/>
       </geometry>
-      <material name="grey"/>
+      <xacro:material_fanuc_grey />
     </visual>
     <collision>

File: src/testbed/safe_energetics_testbed/urdf/m20id35.xacro (robot description, xacro)
@@ -1,8 +1,8 @@
-<?xml version="1.0" ?>
-<robot name="abb_irb6640_180_255" xmlns:xacro="http://ros.org/wiki/xacro">
+<?xml version="1.0"?>
+<robot name="fanuc_m20id35" xmlns:xacro="http://wiki.ros.org/xacro">
   <xacro:include filename="$(find fanuc_m20id35_support)/urdf/fanuc_common_materials.xacro"/>
-  <xacro:include filename="$(find rpi_abb_irb6640_180_255_support)/urdf/irb6640_180_255_fixed_macro.xacro"/>
-  <xacro:abb_irb6640_180_255 prefix="abb_"/>
-  <link name="abb_base_plate">
+  <xacro:include filename="$(find fanuc_m20id35_support)/urdf/m20id35_macro.xacro"/>
+  <xacro:fanuc_m20id35 prefix="fanuc_"/>
+  <link name="fanuc_base_plate">
     <visual>
       <origin rpy="0 0 0" xyz="0 0 0.0127"/>
@@ -19,7 +19,7 @@
     </collision>
   </link>
-  <joint name="abb_base_plate" type="fixed">
-    <parent link="abb_base_plate"/>
-    <child link="abb_base_link"/>
+  <joint name="fanuc_base_plate" type="fixed">
+    <parent link="fanuc_base_plate"/>
+    <child link="fanuc_base_link"/>
     <origin rpy="0 0 0" xyz="0 0 .0254"/>
   </joint>

File: src/testbed/safe_energetics_testbed/urdf/m710ic45m.xacro (robot description, xacro)
@@ -1,4 +1,5 @@
 <?xml version="1.0"?>
 <robot name="fanuc_m710ic45m" xmlns:xacro="http://wiki.ros.org/xacro">
+  <xacro:include filename="$(find fanuc_m20id35_support)/urdf/fanuc_common_materials.xacro"/>
   <xacro:include filename="$(find fanuc_m710ic_support)/urdf/m710ic45m_macro.xacro"/>
   <xacro:fanuc_m710ic45m prefix="fanuc_"/>
@@ -9,5 +10,5 @@
         <box size="0.9144 0.9144 0.0254"/>
       </geometry>
-      <material name="grey"/>
+      <xacro:material_fanuc_grey />
     </visual>
     <collision>

File: src/testbed/safe_energetics_testbed/urdf/safe_energetics_testbed.xacro (robot description, xacro)
@@ -1,7 +1,9 @@
 <?xml version="1.0"?>
 <robot name="safe_energetics_testbed" xmlns:xacro="http://ros.org/wiki/xacro">
+  <xacro:include filename="$(find fanuc_m20id35_support)/urdf/fanuc_common_materials.xacro"/>
   <!-- <xacro:include filename="$(find safe_energetics_testbed)/urdf/irb6640_180_255.xacro"/> -->
   <xacro:include filename="$(find safe_energetics_testbed)/urdf/irb6640_180_255_fixed.xacro"/>
-  <xacro:include filename="$(find safe_energetics_testbed)/urdf/m710ic45m.xacro"/>
+  <!-- <xacro:include filename="$(find safe_energetics_testbed)/urdf/m710ic45m.xacro"/> -->
+  <xacro:include filename="$(find safe_energetics_testbed)/urdf/m20id35.xacro"/>
   <xacro:include filename="$(find safe_energetics_testbed)/urdf/cage.xacro"/>
   <xacro:include filename="$(find safe_energetics_testbed)/urdf/cabinet.xacro"/>
@@ -13,5 +15,5 @@
       <origin xyz="1 0 -.005"/>
       <geometry><box size="8 8 0.01"/></geometry>
-      <material name="grey"/>
+      <xacro:material_fanuc_grey />
     </visual>
     <collision name="collision">
