Commit message: fix ABB robot in cage

File: src/testbed/safe_energetics_testbed/urdf/safe_energetics_testbed.xacro (robot description, xacro)
@@ -1,5 +1,6 @@
 <?xml version="1.0"?>
 <robot name="safe_energetics_testbed" xmlns:xacro="http://ros.org/wiki/xacro">
-  <xacro:include filename="$(find safe_energetics_testbed)/urdf/irb6640_180_255.xacro"/>
+  <!-- <xacro:include filename="$(find safe_energetics_testbed)/urdf/irb6640_180_255.xacro"/> -->
+  <xacro:include filename="$(find safe_energetics_testbed)/urdf/irb6640_180_255_fixed.xacro"/>
   <xacro:include filename="$(find safe_energetics_testbed)/urdf/m710ic45m.xacro"/>
   <xacro:include filename="$(find safe_energetics_testbed)/urdf/cage.xacro"/>
@@ -47,5 +48,5 @@
     <child link="cabinet_base_plate"/>
     <parent link="world"/>
-    <origin rpy="0 0 1.5708" xyz="3.0 0.75 0"/>
+    <origin rpy="0 0 0" xyz="1.5 -1. 0"/>
   </joint>
   <joint name="hopper_long_to_cage" type="fixed">

Commit message: adjust floor plan

File: src/testbed/safe_energetics_testbed/urdf/safe_energetics_testbed.xacro (robot description, xacro)
@@ -28,9 +28,4 @@
     <origin rpy="0 0 0" xyz="0 0 0"/>
   </joint>
-  <joint name="fanuc_robot_to_world" type="fixed">
-    <child link="fanuc_base_plate"/>
-    <parent link="world"/>
-    <origin rpy="0 0 0" xyz="1.5 0.75 0"/>
-  </joint>
   <joint name="cage_to_world" type="fixed">
     <parent link="world"/>
@@ -47,13 +42,18 @@
     <origin rpy="-3.0901665893944226 0.020179445742952443 0.05637854407723496" xyz="0.22644675 -2.46050185  3.44552755"/>
   </joint> -->
+  <joint name="fanuc_robot_to_world" type="fixed">
+    <child link="fanuc_base_plate"/>
+    <parent link="world"/>
+    <origin rpy="0 0 -1.57079" xyz="2.0 2.0 0"/>
+  </joint>
   <joint name="cabinet_to_world" type="fixed">
     <child link="cabinet_base_plate"/>
     <parent link="world"/>
-    <origin rpy="0 0 0" xyz="1.5 -1. 0"/>
+    <origin rpy="0 0 1.57079" xyz="3.2 2.0 0"/>
   </joint>
-  <joint name="hopper_long_to_cage" type="fixed">
+  <joint name="hopper_long_to_world" type="fixed">
     <child link="hopper_long_base_plate"/>
-    <parent link="cage_base_link"/>
-    <origin rpy="0 0 0" xyz="1.0 2.2 0"/>  <!-- x= 0.678, y= 67 inch = 1.7018 m -->
+    <parent link="world"/>
+    <origin rpy="0 0 0" xyz="0.8 1.4945 -0.6096"/>  <!-- x= 0.678, y= 67 inch = 1.7018 m, z = -2ft = -0.6096 m  -->
   </joint>
   <joint name="hopper_short_to_hopper_long" type="fixed">

Commit message: Import OPW kinematics plugin

File: src/testbed/safe_energetics_testbed/urdf/safe_energetics_testbed.xacro (robot description, xacro)
@@ -31,5 +31,5 @@
     <parent link="world"/>
     <child link="cage_base_link"/>
-    <origin rpy="0 0 -1.57079" xyz="-1.282 3.271 0"/>
+    <origin rpy="0 0 -1.57079632679" xyz="-1.282 3.271 0"/>
   </joint>
   <joint name="floor_to_world" type="fixed">
@@ -45,10 +45,10 @@
     <child link="fanuc_base_plate"/>
     <parent link="world"/>
-    <origin rpy="0 0 -1.57079" xyz="2.0 2.0 0"/>
+    <origin rpy="0 0 -1.57079632679" xyz="2.0 2.0 0"/>
   </joint>
   <joint name="cabinet_to_world" type="fixed">
     <child link="cabinet_base_plate"/>
     <parent link="world"/>
-    <origin rpy="0 0 1.57079" xyz="3.2 2.0 0"/>
+    <origin rpy="0 0 1.57079632679" xyz="3.2 2.0 0"/>
   </joint>
   <joint name="hopper_long_to_world" type="fixed">
