Commit message: Add moveit demo package for moveit coding

File: src/testbed/fanuc_m20id35_support/urdf/m20id35_macro.xacro (robot description, xacro)
@@ -153,5 +153,6 @@
     <link name="${prefix}tool0" />
     <joint name="${prefix}link_6-tool0" type="fixed">
-      <origin xyz="0 0 0" rpy="${pi} ${-pi/2.0} 0" />
+      <!-- <origin xyz="0.1 0 0" rpy="${pi} ${-pi/2.0} 0" /> -->
+      <origin xyz="0.1 0 0" rpy="${pi/2.0} 0 ${pi/2.0}" />
       <parent link="${prefix}flange" />
       <child link="${prefix}tool0" />

File: src/testbed/safe_energetics_testbed/urdf/hopper_long.xacro (robot description, xacro)
@@ -3,4 +3,16 @@
   <xacro:include filename="$(find hopper_long)/urdf/hopper_long_macro.xacro"/>
   <xacro:hopper_long prefix=""/>
+  <xacro:property name="h_offset" value="0.1" />
+  <xacro:property name="h_hopper" value="2.286" /> <!-- 82 inch = 2.0828 m, 90 inch = 2.286 m -->
+  <xacro:property name="r_hopper" value="0.25" />
+  <xacro:property name="theta" value="${-45.0/180.0*pi}" /> <!-- rotation around z axis angle (rad)  -->
+  <!-- Pouring point xyz -->
+  <xacro:property name="x_pouring_point" value="${r_hopper * cos(theta)}" />
+  <xacro:property name="y_pouring_point" value="${r_hopper * sin(theta)}" />
+  <xacro:property name="z_pouring_point" value="${h_hopper + h_offset}" />
+  <!-- Pouring point RPY -->
+  <xacro:property name="R_pouring_point" value="${90.0/180.0*pi}" />
+  <xacro:property name="P_pouring_point" value="${0.0/180.0*pi}" />
+  <xacro:property name="Y_pouring_point" value="${theta}" />
   <link name="hopper_long_base_plate">
     <!-- <visual>
@@ -18,4 +30,6 @@
     </collision> -->
   </link>
+  <link name="hopper_long_pouring_point">
+  </link>
   <joint name="hopper_long_base_plate" type="fixed">
     <parent link="hopper_long_base_plate"/>
@@ -25,3 +39,8 @@
     <origin rpy="0 0 0" xyz="0 0 0"/>
   </joint>
+  <joint name="hopper_long_pouring_point" type="fixed">
+    <parent link="hopper_long_base_link"/>
+    <child link="hopper_long_pouring_point"/>
+    <origin xyz="${x_pouring_point} ${y_pouring_point} ${z_pouring_point}" rpy="${R_pouring_point} ${P_pouring_point} ${Y_pouring_point}"/>
+  </joint>
 </robot>

File: src/testbed/safe_energetics_testbed/urdf/hopper_short.xacro (robot description, xacro)
@@ -3,4 +3,16 @@
   <xacro:include filename="$(find hopper_short)/urdf/hopper_short_macro.xacro"/>
   <xacro:hopper_short prefix=""/>
+  <xacro:property name="h_offset" value="0.1" />
+  <xacro:property name="h_hopper" value="2.0828" /> <!-- 82 inch = 2.0828 m -->
+  <xacro:property name="r_hopper" value="0.25" />
+  <xacro:property name="theta" value="${-45.0/180.0*pi}" /> <!-- rotation around z axis angle (rad)  -->
+  <!-- Pouring point xyz -->
+  <xacro:property name="x_pouring_point" value="${r_hopper * cos(theta)}" />
+  <xacro:property name="y_pouring_point" value="${r_hopper * sin(theta)}" />
+  <xacro:property name="z_pouring_point" value="${h_hopper + h_offset}" />
+  <!-- Pouring point RPY -->
+  <xacro:property name="R_pouring_point" value="${90.0/180.0*pi}" />
+  <xacro:property name="P_pouring_point" value="${0.0/180.0*pi}" />
+  <xacro:property name="Y_pouring_point" value="${theta}" />
   <link name="hopper_short_base_plate">
     <!-- <visual>
@@ -18,4 +30,6 @@
     </collision> -->
   </link>
+  <link name="hopper_short_pouring_point">
+  </link>
   <joint name="hopper_short_base_plate" type="fixed">
     <parent link="hopper_short_base_plate"/>
@@ -25,3 +39,8 @@
     <origin rpy="0 0 0" xyz="0 0 0"/>
   </joint>
+  <joint name="hopper_short_pouring_point" type="fixed">
+    <parent link="hopper_short_base_link"/>
+    <child link="hopper_short_pouring_point"/>
+    <origin xyz="${x_pouring_point} ${y_pouring_point} ${z_pouring_point}" rpy="${R_pouring_point} ${P_pouring_point} ${Y_pouring_point}"/>
+  </joint>
 </robot>

Commit message: add test code for pouring procedure

File: src/testbed/fanuc_m20id35_support/urdf/m20id35_macro.xacro (robot description, xacro)
@@ -158,4 +158,20 @@
       <child link="${prefix}tool0" />
     </joint>
+    <xacro:property name="h_pouring_box" value="0.129" />
+    <xacro:property name="r_pouring_box" value="0.055" />
+    <!-- 'Pouring box tip' frame: attached to the tool frame -->
+    <link name="${prefix}pouring_box_tip" />
+    <joint name="${prefix}link_6-tool0-pouring_box_tip" type="fixed">
+      <origin xyz="${-r_pouring_box} ${h_pouring_box/2.0} 0" rpy="0 0 0" /> <!-- Based on pouring box (EMATT) specs -->
+      <parent link="${prefix}tool0" />
+      <child link="${prefix}pouring_box_tip" />
+    </joint>
+    <!-- 'Pouring box bottom' frame: attached to the tool frame -->
+    <link name="${prefix}pouring_box_bottom" />
+    <joint name="${prefix}link_6-tool0-pouring_box_bottom" type="fixed">
+      <origin xyz="0. ${-h_pouring_box/2.0} 0." rpy="0 0 0" /> <!-- Based on pouring box (EMATT) specs -->
+      <parent link="${prefix}tool0" />
+      <child link="${prefix}pouring_box_bottom" />
+    </joint>
   </xacro:macro>
 </robot>

File: src/testbed/safe_energetics_testbed/urdf/cabinet.xacro (robot description, xacro)
@@ -3,4 +3,12 @@
   <xacro:include filename="$(find cabinet)/urdf/cabinet_macro.xacro"/>
   <xacro:cabinet prefix=""/>
+  <xacro:property name="h_level_1" value="0.88" />
+  <xacro:property name="h_level_2" value="1.38" /> <!-- 82 inch = 2.0828 m, 90 inch = 2.286 m -->
+  <xacro:property name="distance_x" value="0.15" />
+  <xacro:property name="distance_y" value="0.0" />
+  <!-- Pouring point RPY -->
+  <xacro:property name="R_pouring_point" value="${90.0/180.0*pi}" />
+  <xacro:property name="P_pouring_point" value="${0.0/180.0*pi}" />
+  <xacro:property name="Y_pouring_point" value="${0.0/180.0*pi}" />
   <link name="cabinet_base_plate">
     <!-- <visual>
@@ -25,3 +33,28 @@
     <origin rpy="0 0 0" xyz="0 0 0"/>
   </joint>
+  <!-- Pickup points in the cabinet -->
+  <link name="cabinet_picking_level_1_point_1"></link>
+  <joint name="cabinet_picking_level_1_point_1" type="fixed">
+    <child link="cabinet_picking_level_1_point_1"/>
+    <parent link="cabinet_base_link"/>
+    <origin xyz="${distance_x} ${distance_y} ${h_level_1}" rpy="${R_pouring_point} ${P_pouring_point} ${Y_pouring_point}"/>
+  </joint>
+  <link name="cabinet_picking_level_1_point_2"></link>
+  <joint name="cabinet_picking_level_1_point_2" type="fixed">
+    <child link="cabinet_picking_level_1_point_2"/>
+    <parent link="cabinet_base_link"/>
+    <origin xyz="${-distance_x} ${distance_y} ${h_level_1}" rpy="${R_pouring_point} ${P_pouring_point} ${Y_pouring_point}"/>
+  </joint>
+  <link name="cabinet_picking_level_2_point_1"></link>
+  <joint name="cabinet_picking_level_2_point_1" type="fixed">
+    <child link="cabinet_picking_level_2_point_1"/>
+    <parent link="cabinet_base_link"/>
+    <origin xyz="${distance_x} ${distance_y} ${h_level_2}" rpy="${R_pouring_point} ${P_pouring_point} ${Y_pouring_point}"/>
+  </joint>
+  <link name="cabinet_picking_level_2_point_2"></link>
+  <joint name="cabinet_picking_level_2_point_2" type="fixed">
+    <child link="cabinet_picking_level_2_point_2"/>
+    <parent link="cabinet_base_link"/>
+    <origin xyz="${-distance_x} ${distance_y} ${h_level_2}" rpy="${R_pouring_point} ${P_pouring_point} ${Y_pouring_point}"/>
+  </joint>
 </robot>
